File: EnvOpenPico.sch (KiCad schematic (older format))
At the start: 40 parts, among them J1 USB_B_Micro, J2 Conn_01x02, J3 Conn_02x18_Odd_Even, J4 Conn_02x18_Odd_Even, J5 Conn_01x03_Male, U1 NCP1117-3.3_SOT223, U2 W25Q16JVSSIQ, U3 RP2040, Y1 ABLS-12.000MHZ-B4-T

Commit message: more progress bits
Parts:
- removed C13, C14, C15, C16: 100n, Capacitor_SMD:C_0402_1005Metric, symbol Device:C
- D3: footprint LED_SMD:LED_0805_2012Metric -> LED_SMD:LED_0402_1005Metric
- R8: footprint Resistor_SMD:R_0805_2012Metric -> Resistor_SMD:R_0402_1005Metric
Connections:
- wire segments 205 -> 188
Changed lines of the file:
@@
 Connection ~ 7000 3200
-$Comp
-L Device:C C9
-U 1 1 5EEEE897
-P 8800 2600
-F 0 "C9" H 8915 2646 50  0000 L CNN
-F 1 "100n" H 8915 2555 50  0000 L CNN
-F 2 "Capacitor_SMD:C_0402_1005Metric" H 8838 2450 50  0001 C CNN
-F 3 "~" H 8800 2600 50  0001 C CNN
-	1    8800 2600
-	1    0    0    -1
-$EndComp
-$Comp
-L Device:C C11
-U 1 1 5EEF00BB
-P 9250 2600
-F 0 "C11" H 9365 2646 50  0000 L CNN
-F 1 "100n" H 9365 2555 50  0000 L CNN
-F 2 "Capacitor_SMD:C_0402_1005Metric" H 9288 2450 50  0001 C CNN
-F 3 "~" H 9250 2600 50  0001 C CNN
-	1    9250 2600
-	1    0    0    -1
-$EndComp
-$Comp
-L Device:C C12
-U 1 1 5EEF0473
-P 9700 2600
-F 0 "C12" H 9815 2646 50  0000 L CNN
-F 1 "100n" H 9815 2555 50  0000 L CNN
-F 2 "Capacitor_SMD:C_0402_1005Metric" H 9738 2450 50  0001 C CNN
-F 3 "~" H 9700 2600 50  0001 C CNN
-	1    9700 2600
-	1    0    0    -1
-$EndComp
-$Comp
-L Device:C C13
-U 1 1 5EEF0994
-P 10150 2600
-F 0 "C13" H 10265 2646 50  0000 L CNN
-F 1 "100n" H 10265 2555 50  0000 L CNN
-F 2 "Capacitor_SMD:C_0402_1005Metric" H 10188 2450 50  0001 C CNN
-F 3 "~" H 10150 2600 50  0001 C CNN
-	1    10150 2600
-	1    0    0    -1
-$EndComp
-$Comp
-L Device:C C14
-U 1 1 5EEF89B3
-P 10600 2600
-F 0 "C14" H 10715 2646 50  0000 L CNN
-F 1 "100n" H 10715 2555 50  0000 L CNN
-F 2 "Capacitor_SMD:C_0402_1005Metric" H 10638 2450 50  0001 C CNN
-F 3 "~" H 10600 2600 50  0001 C CNN
-	1    10600 2600
-	1    0    0    -1
-$EndComp
-$Comp
-L Device:C C15
-U 1 1 5EEF89BD
-P 11050 2600
-F 0 "C15" H 11165 2646 50  0000 L CNN
-F 1 "100n" H 11165 2555 50  0000 L CNN
-F 2 "Capacitor_SMD:C_0402_1005Metric" H 11088 2450 50  0001 C CNN
-F 3 "~" H 11050 2600 50  0001 C CNN
-	1    11050 2600
-	1    0    0    -1
-$EndComp
-$Comp
-L Device:C C16
-U 1 1 5EEF89C7
-P 11500 2600
-F 0 "C16" H 11615 2646 50  0000 L CNN
-F 1 "100n" H 11615 2555 50  0000 L CNN
-F 2 "Capacitor_SMD:C_0402_1005Metric" H 11538 2450 50  0001 C CNN
-F 3 "~" H 11500 2600 50  0001 C CNN
-	1    11500 2600
-	1    0    0    -1
-$EndComp
 $Comp
 L Device:C C6
@@
 $EndComp
 Wire Wire Line
-	11500 2450 11500 2400
-Wire Wire Line
-	11050 2450 11050 2400
-Connection ~ 11050 2400
-Wire Wire Line
-	11050 2400 11500 2400
-Wire Wire Line
-	10600 2450 10600 2400
-Connection ~ 10600 2400
-Wire Wire Line
-	10600 2400 11050 2400
-Wire Wire Line
-	10150 2450 10150 2400
-Connection ~ 10150 2400
-Wire Wire Line
-	10150 2400 10600 2400
-Wire Wire Line
 	9700 2450 9700 2400
-Connection ~ 9700 2400
-Wire Wire Line
-	9700 2400 10150 2400
 Wire Wire Line
 	9250 2450 9250 2400
@@
 Wire Wire Line
 	8800 2400 9250 2400
-$Comp
-L power:GND #PWR023
-U 1 1 5EF621A6
-P 11500 2900
-F 0 "#PWR023" H 11500 2650 50  0001 C CNN
-F 1 "GND" H 11505 2727 50  0000 C CNN
-F 2 "" H 11500 2900 50  0001 C CNN
-F 3 "" H 11500 2900 50  0001 C CNN
-	1    11500 2900
-	1    0    0    -1
-$EndComp
 Wire Wire Line
 	8800 2750 8800 2850
@@
 Wire Wire Line
 	9700 2750 9700 2850
-Connection ~ 9700 2850
 Wire Wire Line
 	9700 2850 9250 2850
-Wire Wire Line
-	10150 2750 10150 2850
-Connection ~ 10150 2850
-Wire Wire Line
-	10150 2850 9700 2850
-Wire Wire Line
-	10600 2750 10600 2850
-Connection ~ 10600 2850
-Wire Wire Line
-	10600 2850 10150 2850
-Wire Wire Line
-	11050 2750 11050 2850
-Wire Wire Line
-	11050 2850 10600 2850
-Wire Wire Line
-	11500 2750 11500 2850
 Wire Wire Line
 	6650 3050 6650 3000
@@
 $EndComp
 NoConn ~ 1600 2150
-Wire Wire Line
-	11050 2850 11500 2850
-Connection ~ 11050 2850
-Connection ~ 11500 2850
-Wire Wire Line
-	11500 2850 11500 2900
 $Comp
 L Device:R R5
@@
 F 0 "R8" V 14293 7600 50  0000 C CNN
 F 1 "R470" V 14384 7600 50  0000 C CNN
-F 2 "Resistor_SMD:R_0805_2012Metric" V 14430 7600 50  0001 C CNN
+F 2 "Resistor_SMD:R_0402_1005Metric" V 14430 7600 50  0001 C CNN
 F 3 "~" H 14500 7600 50  0001 C CNN
 	1    14500 7600
@@
 F 0 "D3" H 14750 7350 50  0000 C CNN
 F 1 "GPIO25 LED" H 14600 7450 50  0000 C CNN
-F 2 "LED_SMD:LED_0805_2012Metric" H 14800 7600 50  0001 C CNN
+F 2 "LED_SMD:LED_0402_1005Metric" H 14800 7600 50  0001 C CNN
 F 3 "~" H 14800 7600 50  0001 C CNN
 	1    14800 7600
@@
 Wire Wire Line
 	14100 5200 14550 5200
+$Comp
+L Device:C C12
+U 1 1 5EEF0473
+P 9700 2600
+F 0 "C12" H 9815 2646 50  0000 L CNN
+F 1 "100n" H 9815 2555 50  0000 L CNN
+F 2 "Capacitor_SMD:C_0402_1005Metric" H 9738 2450 50  0001 C CNN
+F 3 "~" H 9700 2600 50  0001 C CNN
+	1    9700 2600
+	1    0    0    -1
+$EndComp
+$Comp
+L Device:C C11
+U 1 1 5EEF00BB
+P 9250 2600
+F 0 "C11" H 9365 2646 50  0000 L CNN
+F 1 "100n" H 9365 2555 50  0000 L CNN
+F 2 "Capacitor_SMD:C_0402_1005Metric" H 9288 2450 50  0001 C CNN
+F 3 "~" H 9250 2600 50  0001 C CNN
+	1    9250 2600
+	1    0    0    -1
+$EndComp
+$Comp
+L Device:C C9
+U 1 1 5EEEE897
+P 8800 2600
+F 0 "C9" H 8915 2646 50  0000 L CNN
+F 1 "100n" H 8915 2555 50  0000 L CNN
+F 2 "Capacitor_SMD:C_0402_1005Metric" H 8838 2450 50  0001 C CNN
+F 3 "~" H 8800 2600 50  0001 C CNN
+	1    8800 2600
+	1    0    0    -1
+$EndComp
+$Comp
+L power:GND #PWR0105
+U 1 1 608B0015
+P 9700 2850
+F 0 "#PWR0105" H 9700 2600 50  0001 C CNN
+F 1 "GND" H 9705 2677 50  0000 C CNN
+F 2 "" H 9700 2850 50  0001 C CNN
+F 3 "" H 9700 2850 50  0001 C CNN
+	1    9700 2850
+	1    0    0    -1
+$EndComp
+Connection ~ 9700 2850
 $EndSCHEMATC

Commit message: did more things!
Parts:
- J2: footprint Connector_PinHeader_2.54mm:PinHeader_1x02_P2.54mm_Vertical -> Connector_PinHeader_1.00mm:PinHeader_1x02_P1.00mm_Vertical
Changed lines of the file:
@@
 F 0 "J2" H 1100 5100 50  0000 C CNN
 F 1 "Conn_01x02" H 1100 4700 50  0000 C CNN
-F 2 "Connector_PinHeader_2.54mm:PinHeader_1x02_P2.54mm_Vertical" H 1050 4950 50  0001 C CNN
+F 2 "Connector_PinHeader_1.00mm:PinHeader_1x02_P1.00mm_Vertical" H 1050 4950 50  0001 C CNN
 F 3 "~" H 1050 4950 50  0001 C CNN
 	1    1050 4950

Commit message: progress+1
Parts:
- C1, C4: footprint Capacitor_SMD:C_0805_2012Metric -> Capacitor_SMD:C_0402_1005Metric
Changed lines of the file:
@@
 F 0 "C1" H 2415 1996 50  0000 L CNN
 F 1 "10u" H 2415 1905 50  0000 L CNN
-F 2 "Capacitor_SMD:C_0805_2012Metric" H 2338 1800 50  0001 C CNN
+F 2 "Capacitor_SMD:C_0402_1005Metric" H 2338 1800 50  0001 C CNN
 F 3 "~" H 2300 1950 50  0001 C CNN
 	1    2300 1950
@@
 F 0 "C4" H 3815 1996 50  0000 L CNN
 F 1 "10u" H 3815 1905 50  0000 L CNN
-F 2 "Capacitor_SMD:C_0805_2012Metric" H 3738 1800 50  0001 C CNN
+F 2 "Capacitor_SMD:C_0402_1005Metric" H 3738 1800 50  0001 C CNN
 F 3 "~" H 3700 1950 50  0001 C CNN
 	1    3700 1950

Commit message: Redesign
I need sleep.
Parts:
- removed C9: 100n, Capacitor_SMD:C_0402_1005Metric, symbol Device:C
- removed R6: R200, Resistor_SMD:R_0805_2012Metric, symbol Device:R
- removed R7: R1, Resistor_SMD:R_0805_2012Metric, symbol Device:R
- added C13, C14, C15: 100n, Capacitor_SMD:C_0402_1005Metric, symbol Device:C
- U2: footprint W25Q16JVSSIQ:SOIC127P790X216-8N -> Package_SO:SOIC-8_5.23x5.23mm_P1.27mm
Connections:
- wire segments 188 -> 191
Changed lines of the file:
@@
 	9250 2400 9700 2400
 Wire Wire Line
-	8800 2450 8800 2400
-Connection ~ 8800 2400
-Wire Wire Line
-	8800 2400 9250 2400
-Wire Wire Line
-	8800 2750 8800 2850
-Wire Wire Line
 	9250 2750 9250 2850
-Connection ~ 9250 2850
-Wire Wire Line
-	9250 2850 8800 2850
 Wire Wire Line
 	9700 2750 9700 2850
@@
 	8450 3000 8450 3200
 Wire Wire Line
-	8450 2400 8800 2400
-Wire Wire Line
 	8450 2350 8450 2400
 Connection ~ 8450 2400
-Wire Wire Line
-	8450 2400 8450 2800
 $Comp
 L Switch:SW_Push J2
@@
 	0    -1   -1   0
 $EndComp
-$Comp
-L Device:R R7
-U 1 1 60B82AF4
-P 7900 2800
-F 0 "R7" V 7800 2800 50  0000 C CNN
-F 1 "R1" V 8000 2800 50  0000 C CNN
-F 2 "Resistor_SMD:R_0805_2012Metric" V 7830 2800 50  0001 C CNN
-F 3 "~" H 7900 2800 50  0001 C CNN
-	1    7900 2800
-	0    1    1    0
-$EndComp
-Wire Wire Line
-	8050 2800 8450 2800
-Connection ~ 8450 2800
-Wire Wire Line
-	8450 2800 8450 3000
-Text Label 7850 2550 0    50   ~ 0
-ADC_VREF
-Wire Wire Line
-	7750 2550 7850 2550
-Wire Wire Line
-	7750 2550 7750 2800
-Wire Wire Line
-	7750 2550 7750 2450
-Connection ~ 7750 2550
-$Comp
-L Device:R R6
-U 1 1 60BB7E33
-P 7750 2300
-F 0 "R6" H 7820 2346 50  0000 L CNN
-F 1 "R200" H 7820 2255 50  0000 L CNN
-F 2 "Resistor_SMD:R_0805_2012Metric" V 7680 2300 50  0001 C CNN
-F 3 "~" H 7750 2300 50  0001 C CNN
-	1    7750 2300
-	1    0    0    -1
-$EndComp
-$Comp
-L power:+3V3 #PWR022
-U 1 1 60BB8A40
-P 7750 2150
-F 0 "#PWR022" H 7750 2000 50  0001 C CNN
-F 1 "+3V3" H 7765 2323 50  0000 C CNN
-F 2 "" H 7750 2150 50  0001 C CNN
-F 3 "" H 7750 2150 50  0001 C CNN
-	1    7750 2150
-	1    0    0    -1
-$EndComp
 Text Label 14100 5200 0    39   ~ 0
 ADC_VREF
@@
 F 0 "U2" H 3400 4400 50  0000 C CNN
 F 1 "W25Q16JVSSIQ" H 3400 4550 50  0000 C CNN
-F 2 "W25Q16JVSSIQ:SOIC127P790X216-8N" H 3400 5150 50  0001 L BNN
+F 2 "Package_SO:SOIC-8_5.23x5.23mm_P1.27mm" H 3400 5150 50  0001 L BNN
 F 3 "" H 3400 5150 50  0001 L BNN
 F 4 "Unavailable" H 3400 5150 50  0001 L BNN "AVAILABILITY"
@@
 	1    0    0    -1
 $EndComp
-$Comp
-L Device:C C9
-U 1 1 5EEEE897
-P 8800 2600
-F 0 "C9" H 8915 2646 50  0000 L CNN
-F 1 "100n" H 8915 2555 50  0000 L CNN
-F 2 "Capacitor_SMD:C_0402_1005Metric" H 8838 2450 50  0001 C CNN
-F 3 "~" H 8800 2600 50  0001 C CNN
-	1    8800 2600
-	1    0    0    -1
-$EndComp
-$Comp
-L power:GND #PWR0105
-U 1 1 608B0015
-P 9700 2850
-F 0 "#PWR0105" H 9700 2600 50  0001 C CNN
-F 1 "GND" H 9705 2677 50  0000 C CNN
-F 2 "" H 9700 2850 50  0001 C CNN
-F 3 "" H 9700 2850 50  0001 C CNN
-	1    9700 2850
-	1    0    0    -1
-$EndComp
 Connection ~ 9700 2850
+Wire Wire Line
+	11000 2450 11000 2400
+Wire Wire Line
+	10550 2450 10550 2400
+Connection ~ 10550 2400
+Wire Wire Line
+	10550 2400 11000 2400
+Wire Wire Line
+	10100 2450 10100 2400
+Connection ~ 10100 2400
+Wire Wire Line
+	10100 2400 10550 2400
+Wire Wire Line
+	10100 2750 10100 2850
+Wire Wire Line
+	10550 2750 10550 2850
+Connection ~ 10550 2850
+Wire Wire Line
+	10550 2850 10100 2850
+Wire Wire Line
+	11000 2750 11000 2850
+Wire Wire Line
+	11000 2850 10550 2850
+$Comp
+L Device:C C15
+U 1 1 608F1359
+P 11000 2600
+F 0 "C15" H 11115 2646 50  0000 L CNN
+F 1 "100n" H 11115 2555 50  0000 L CNN
+F 2 "Capacitor_SMD:C_0402_1005Metric" H 11038 2450 50  0001 C CNN
+F 3 "~" H 11000 2600 50  0001 C CNN
+	1    11000 2600
+	1    0    0    -1
+$EndComp
+$Comp
+L Device:C C14
+U 1 1 608F135F
+P 10550 2600
+F 0 "C14" H 10665 2646 50  0000 L CNN
+F 1 "100n" H 10665 2555 50  0000 L CNN
+F 2 "Capacitor_SMD:C_0402_1005Metric" H 10588 2450 50  0001 C CNN
+F 3 "~" H 10550 2600 50  0001 C CNN
+	1    10550 2600
+	1    0    0    -1
+$EndComp
+$Comp
+L Device:C C13
+U 1 1 608F1365
+P 10100 2600
+F 0 "C13" H 10215 2646 50  0000 L CNN
+F 1 "100n" H 10215 2555 50  0000 L CNN
+F 2 "Capacitor_SMD:C_0402_1005Metric" H 10138 2450 50  0001 C CNN
+F 3 "~" H 10100 2600 50  0001 C CNN
+	1    10100 2600
+	1    0    0    -1
+$EndComp
+$Comp
+L power:GND #PWR08
+U 1 1 608F136B
+P 11000 2850
+F 0 "#PWR08" H 11000 2600 50  0001 C CNN
+F 1 "GND" H 11005 2677 50  0000 C CNN
+F 2 "" H 11000 2850 50  0001 C CNN
+F 3 "" H 11000 2850 50  0001 C CNN
+	1    11000 2850
+	1    0    0    -1
+$EndComp
+Connection ~ 11000 2850
+Wire Wire Line
+	9700 2400 10100 2400
+Connection ~ 9700 2400
+Wire Wire Line
+	9700 2850 10100 2850
+Connection ~ 10100 2850
+Wire Wire Line
+	8450 2400 8450 3000
+Wire Wire Line
+	8450 2400 9250 2400
 $EndSCHEMATC

Commit message: Swapped Crystal for smaller XO oscillator
+ some general other changes
Parts:
- removed C12: 100n, Capacitor_SMD:C_0402_1005Metric, symbol Device:C
- removed C3: 27p, Capacitor_SMD:C_0402_1005Metric, symbol Device:C
- removed C8: 1u, Capacitor_SMD:C_0402_1005Metric, symbol Device:C
- removed R5: 1k, Capacitor_SMD:C_0402_1005Metric, symbol Device:R
- removed Y1: ABLS-12.000MHZ-B4-T, Crystal:Crystal_SMD_5032-2Pin_5.0x3.2mm, symbol Device:Crystal
- added X1: XO32, Crystal:Crystal_SMD_SeikoEpson_TSX3225-4Pin_3.2x2.5mm, symbol Oscillator:XO32
- C17: footprint Capacitor_SMD:C_0805_2012Metric -> Capacitor_SMD:C_0201_0603Metric
- C2: value 27p -> 15p
Connections:
- net labels added: +3.3V
- wire segments 191 -> 175
Other:
- note added: "Intentionally left floating"
- note added: "also left floating so the chip is enabled"
- moved on the sheet: C2
Changed lines of the file:
@@
-	1    0    0    -1
-$EndComp
-$Comp
-L Device:C C2
-U 1 1 5ED96B87
-P 2000 8600
-F 0 "C2" H 2115 8646 50  0000 L CNN
-F 1 "27p" H 2115 8555 50  0000 L CNN
-F 2 "Capacitor_SMD:C_0402_1005Metric" H 2038 8450 50  0001 C CNN
-F 3 "~" H 2000 8600 50  0001 C CNN
-	1    2000 8600
-	0    1    1    0
-$EndComp
-$Comp
-L Device:C C3
-U 1 1 5ED98685
-P 2000 9000
-F 0 "C3" H 2115 9046 50  0000 L CNN
-F 1 "27p" H 2115 8955 50  0000 L CNN
-F 2 "Capacitor_SMD:C_0402_1005Metric" H 2038 8850 50  0001 C CNN
-F 3 "~" H 2000 9000 50  0001 C CNN
-	1    2000 9000
-	0    1    1    0
-$EndComp
-$Comp
-L power:GND #PWR06
-U 1 1 5ED9B1CB
-P 1750 9100
-F 0 "#PWR06" H 1750 8850 50  0001 C CNN
-F 1 "GND" H 1755 8927 50  0000 C CNN
-F 2 "" H 1750 9100 50  0001 C CNN
-F 3 "" H 1750 9100 50  0001 C CNN
-	1    1750 9100
 	1    0    0    -1
 $EndComp
@@
 Wire Wire Line
 	6550 6000 6000 6000
-Wire Wire Line
-	1850 8600 1750 8600
-Wire Wire Line
-	1750 8600 1750 9000
-Wire Wire Line
-	1850 9000 1750 9000
-Connection ~ 1750 9000
-Wire Wire Line
-	1750 9000 1750 9100
-Wire Wire Line
-	2150 9000 2600 9000
-Wire Wire Line
-	2150 8600 2600 8600
-Wire Wire Line
-	2600 8650 2600 8600
-Wire Wire Line
-	2600 8950 2600 9000
-Connection ~ 2600 9000
-Wire Wire Line
-	2600 9000 3150 9000
 Wire Wire Line
 	6000 4600 6550 4600
@@
 $EndComp
 $Comp
-L Device:C C8
-U 1 1 5EF07987
-P 6650 3200
-F 0 "C8" H 6765 3246 50  0000 L CNN
-F 1 "1u" H 6765 3155 50  0000 L CNN
-F 2 "Capacitor_SMD:C_0402_1005Metric" H 6688 3050 50  0001 C CNN
-F 3 "~" H 6650 3200 50  0001 C CNN
-	1    6650 3200
-	1    0    0    -1
-$EndComp
-$Comp
 L Device:C C10
 U 1 1 5EF08170
@@
 $EndComp
 Wire Wire Line
-	9700 2450 9700 2400
-Wire Wire Line
 	9250 2450 9250 2400
 Connection ~ 9250 2400
 Wire Wire Line
-	9250 2400 9700 2400
-Wire Wire Line
 	9250 2750 9250 2850
-Wire Wire Line
-	9700 2750 9700 2850
-Wire Wire Line
-	9700 2850 9250 2850
-Wire Wire Line
-	6650 3050 6650 3000
-Wire Wire Line
-	6650 3000 7000 3000
-Connection ~ 7000 3000
-Wire Wire Line
-	7000 3000 7000 3200
 Wire Wire Line
 	8800 3050 8800 3000
@@
 Connection ~ 7000 2400
 Wire Wire Line
-	7000 2400 7000 3000
-Wire Wire Line
 	6650 2450 6650 2400
 Connection ~ 6650 2400
@@
 	6650 2400 7000 2400
 Wire Wire Line
-	6650 3350 6650 3400
-Wire Wire Line
 	8800 3350 8800 3400
-$Comp
-L power:GND #PWR013
-U 1 1 5F00AFBA
-P 6650 3400
-F 0 "#PWR013" H 6650 3150 50  0001 C CNN
-F 1 "GND" H 6655 3227 50  0000 C CNN
-F 2 "" H 6650 3400 50  0001 C CNN
-F 3 "" H 6650 3400 50  0001 C CNN
-	1    6650 3400
-	1    0    0    -1
-$EndComp
 $Comp
 L power:GND #PWR018
@@
 $EndComp
 NoConn ~ 1600 2150
-$Comp
-L Device:R R5
-U 1 1 5F0D8EBF
-P 3300 9000
-F 0 "R5" V 3093 9000 50  0000 C CNN
-F 1 "1k" V 3184 9000 50  0000 C CNN
-F 2 "Capacitor_SMD:C_0402_1005Metric" V 3230 9000 50  0001 C CNN
-F 3 "~" H 3300 9000 50  0001 C CNN
-	1    3300 9000
-	0    1    1    0
-$EndComp
-$Comp
-L Device:Crystal Y1
-U 1 1 5F0DD35C
-P 2600 8800
-F 0 "Y1" V 2554 8931 50  0000 L CNN
-F 1 "ABLS-12.000MHZ-B4-T" V 2300 8550 50  0000 L CNN
-F 2 "Crystal:Crystal_SMD_5032-2Pin_5.0x3.2mm" H 2600 8800 50  0001 C CNN
-F 3 "~" H 2600 8800 50  0001 C CNN
-	1    2600 8800
-	0    1    1    0
-$EndComp
 Text Notes 9100 3300 0    50   ~ 0
 Make sure C10 is close to pin 44 of RP2040
@@
 F 0 "C17" H 13515 7246 50  0000 L CNN
 F 1 "10u" H 13515 7155 50  0000 L CNN
-F 2 "Capacitor_SMD:C_0805_2012Metric" H 13438 7050 50  0001 C CNN
+F 2 "Capacitor_SMD:C_0201_0603Metric" H 13438 7050 50  0001 C CNN
 F 3 "~" H 13400 7200 50  0001 C CNN
 	1    13400 7200
@@
 Wire Wire Line
 	13400 7350 13400 7400
-Text Notes 1850 8300 0    197  ~ 39
+Text Notes 1350 7750 0    197  ~ 39
 Crystal
 Text Notes 2150 3600 0    197  ~ 39
@@
 Wire Wire Line
 	13400 6950 13400 7050
-Text Label 3850 8600 2    50   ~ 0
+Text Label 3850 8400 2    50   ~ 0
 XIN
-Text Label 3850 9000 2    50   ~ 0
+Text Label 3900 9000 2    50   ~ 0
 XOUT
 Wire Wire Line
-	2600 8600 3850 8600
-Wire Wire Line
-	3450 9000 3850 9000
-Connection ~ 2600 8600
+	2600 8400 3200 8400
 Text Notes 9950 3950 0    50   ~ 0
 Make sure R3 and R4 are close to RP2040
@@
 	14100 5200 14550 5200
 $Comp
-L Device:C C12
-U 1 1 5EEF0473
-P 9700 2600
-F 0 "C12" H 9815 2646 50  0000 L CNN
-F 1 "100n" H 9815 2555 50  0000 L CNN
-F 2 "Capacitor_SMD:C_0402_1005Metric" H 9738 2450 50  0001 C CNN
-F 3 "~" H 9700 2600 50  0001 C CNN
-	1    9700 2600
-	1    0    0    -1
-$EndComp
-$Comp
 L Device:C C11
 U 1 1 5EEF00BB
@@
 	1    0    0    -1
 $EndComp
-Connection ~ 9700 2850
 Wire Wire Line
 	11000 2450 11000 2400
@@
 $EndComp
 Connection ~ 11000 2850
-Wire Wire Line
-	9700 2400 10100 2400
-Connection ~ 9700 2400
-Wire Wire Line
-	9700 2850 10100 2850
 Connection ~ 10100 2850
 Wire Wire Line
@@
 Wire Wire Line
 	8450 2400 9250 2400
+$Comp
+L Oscillator:XO32 X1
+U 1 1 60894744
+P 2600 8700
+F 0 "X1" V 2250 8550 50  0000 L CNN
+F 1 "XO32" V 2350 8450 50  0000 L CNN
+F 2 "Crystal:Crystal_SMD_SeikoEpson_TSX3225-4Pin_3.2x2.5mm" H 3300 8350 50  0001 C CNN
+F 3 "http://cdn-reichelt.de/documents/datenblatt/B400/XO32.pdf" H 2500 8700 50  0001 C CNN
+	1    2600 8700
+	0    -1   -1   0
+$EndComp
+$Comp
+L power:GND #PWR0105
+U 1 1 608B9527
+P 2900 8700
+F 0 "#PWR0105" H 2900 8450 50  0001 C CNN
+F 1 "GND" V 2905 8572 50  0000 R CNN
+F 2 "" H 2900 8700 50  0001 C CNN
+F 3 "" H 2900 8700 50  0001 C CNN
+	1    2900 8700
+	0    -1   -1   0
+$EndComp
+$Comp
+L power:+3.3V #PWR0106
+U 1 1 608B9D1F
+P 2300 8700
+F 0 "#PWR0106" H 2300 8550 50  0001 C CNN
+F 1 "+3.3V" V 2315 8828 50  0000 L CNN
+F 2 "" H 2300 8700 50  0001 C CNN
+F 3 "" H 2300 8700 50  0001 C CNN
+	1    2300 8700
+	0    -1   -1   0
+$EndComp
+$Comp
+L Device:C C2
+U 1 1 5ED96B87
+P 3200 8250
+F 0 "C2" H 3315 8296 50  0000 L CNN
+F 1 "15p" H 3315 8205 50  0000 L CNN
+F 2 "Capacitor_SMD:C_0402_1005Metric" H 3238 8100 50  0001 C CNN
+F 3 "~" H 3200 8250 50  0001 C CNN
+	1    3200 8250
+	1    0    0    -1
+$EndComp
+Connection ~ 3200 8400
+Wire Wire Line
+	3200 8400 3850 8400
+$Comp
+L power:GND #PWR0107
+U 1 1 6097CBA8
+P 3200 8100
+F 0 "#PWR0107" H 3200 7850 50  0001 C CNN
+F 1 "GND" H 3205 7927 50  0000 C CNN
+F 2 "" H 3200 8100 50  0001 C CNN
+F 3 "" H 3200 8100 50  0001 C CNN
+	1    3200 8100
+	-1   0    0    1
+$EndComp
+Wire Wire Line
+	3650 9000 3900 9000
+Text Notes 3450 9100 0    39   ~ 0
+Intentionally left floating
+Text Notes 1750 9200 0    50   ~ 0
+also left floating so the chip is enabled
+Wire Wire Line
+	7000 2400 7000 3200
+Wire Wire Line
+	9250 2850 10100 2850
+Wire Wire Line
+	9250 2400 10100 2400
 $EndSCHEMATC
