File: EnvOpenPico/EnvOpenPico.kicad_pcb (KiCad board)
At the start: 2 copper layers, 21.1 x 51.3 mm, 41 parts, among them J2 SKRKAEE020, J3 2.54mm header 01x20, J4 2.54mm header 01x20, J5 Conn_01x03_Male, U1 TPS63002, U3 RP2040, X1 XO 32 12Mhz 3225 seiko

Commit message: bit of a redesign.
Parts:
- added C16: 100nf 0402, Capacitor_SMD:C_0402_1005Metric, F.Cu at (109.7, 81.9)
- added C18: 100nf 0402, Capacitor_SMD:C_0402_1005Metric, F.Cu at (109.7, 80.7)
- C1: value 10uf 0402 -> 10uf 0603 6.3V; footprint Capacitor_SMD:C_0402_1005Metric -> Capacitor_SMD:C_0603_1608Metric
- FLASH1: footprint Package_SO:SOIJ-8_5.3x5.3mm_P1.27mm -> Package_SON:SON-8-1EP_3x2mm_P0.5mm_EP1.4x1.6mm
- moved C5 6.88 mm to (99.7, 76.7), turned to 90 degrees
- moved R1 5.47 mm to (98.7, 76.7), turned to 90 degrees
- moved TP3 5.24 mm to (106.2, 64.8)
- moved J2 5.06 mm to (99.3, 72.9)
- moved C12 4.42 mm to (104.3, 71.0), turned to 270 degrees
- moved R5 3.63 mm to (105.1, 66.6), turned to 90 degrees
- moved R7 3.20 mm to (106.1, 67.2), turned to 270 degrees
- moved FLASH1 3.09 mm to (100.5, 79.4)
- moved C7 2.45 mm to (103.2, 80.3), turned to 90 degrees
- moved C4 1.73 mm to (109.6, 72.6), turned to 0 degrees
- moved R6 1.65 mm to (101.8, 66.6), turned to 90 degrees
- moved R3 1.34 mm to (104.4, 78.5)
- moved R4 1.34 mm to (105.3, 78.5)
- moved C13 1.33 mm to (110.1, 87.0)
- moved C8 0.93 mm to (104.2, 80.3)
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Routing:
- net Net-(R5-Pad2): track 10.1 -> 1.47 mm, vias 2 -> 0
- net /QSPI_SD3: track 16.0 -> 7.86 mm
- net /QSPI_SCLK: track 14.1 -> 6.73 mm
- net /QSPI_SS: track 18.7 -> 11.7 mm, vias 2 -> 1
- net /QSPI_SD0: track 10.1 -> 4.87 mm
- net +3V3: track 55.3 -> 60.5 mm, vias 4 -> 3
- net USB_D-: track 20.2 -> 15.5 mm, vias 2 -> 3
- net USB_D+: track 20.3 -> 15.7 mm, vias 2 -> 4
- net VBUS: track 1.72 -> 5.94 mm
- net +1V1: track 19.9 -> 15.8 mm, vias 6 -> 5
- net 3V3_EN: track 10.7 -> 14.0 mm, vias 3 -> 1
- net Net-(R6-Pad2): track 3.98 -> 1.48 mm
- net /QSPI_SD1: track 4.51 -> 2.65 mm
- net GND: track 31.8 -> 30.2 mm, vias 21 -> 15
- net Net-(R3-Pad2): track 2.43 -> 3.85 mm
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- added copper zone on F.Cu, net Net-(L1-Pad1)
- added copper zone on F.Cu, net Net-(L1-Pad2)
- removed copper zone on F.Cu, net 3V3_EN
