File: RP2040/EnvOpenPico2040/EnvOpenPico-RP2040.kicad_sch (KiCad schematic)
At the start: 55 parts, among them J1 USB_C_Receptacle_USB2.0, J2 Button, J3 2.54mm header 01x20, J4 2.54mm header 01x20, J5 Conn_01x03_Male, Q1 SI2301B, U1 SOT-23-5 5.5V 3.3V 500mA, U3 RP2040, Y1 3225_4P 12MHz

Commit message: made many corrections to RP2040 pico board, silkscreen, positioning, footprint, any errors I could find.
Parts:
- D1: value 1N4002W -> 1N5817W
- FLASH1: footprint Package_SON:SON-8-1EP_3x2mm_P0.5mm_EP1.4x1.6mm -> Package_SON:Winbond_USON-8-1EP_3x2mm_P0.5mm_EP0.2x1.6mm
Connections:
- no-connect marks 0 -> 2
Other:
- note added: "D1 NEEDS to be 0omh resistor or 1N5817W diode"
- note added: "Power LED is on by default but when GPIO23 is enabled it will be shut off"
- note removed: "D1 NEEDS to be 0omh resistor or 1N4002 diode"
- note removed: "Power LED is on by default but when GPIO24 is enabled it will be shut off"
