File: RP2350/EnvOpenPico2350/EnvOpenPico2350.kicad_pcb (KiCad board)
At the start: 2 copper layers, 21 x 51 mm, 59 parts, among them J1 USB_C_Receptacle_USB2.0, J2 TSA343G00-250J2, J3 2.54mm header 01x20, J4 2.54mm header 01x20, J5 Conn_01x03_Male, Q1 SI2301B, U1 SOT-23-5 5.5V 3.3V 500mA, U3 RP2350A, Y1 3225_4P 12MHz

Commit message: made various corrections and adjustments to the board, generated production files.
Parts:
- D1: value 1N4002W -> 1N5917W
- FLASH1: footprint Package_SON:SON-8-1EP_3x2mm_P0.5mm_EP1.4x1.6mm -> Package_SON:Winbond_USON-8-1EP_3x2mm_P0.5mm_EP0.2x1.6mm
- moved R4 1.07 mm to (105.9, 74.8)
- moved R3 1.02 mm to (104.8, 74.8)
- moved C6 0.55 mm to (105.9, 79.9)
- moved C3 0.52 mm to (105.8, 80.9)
- moved L1 0.17 mm to (105.8, 78.1)
Routing:
- net GND: track 26.0 -> 29.8 mm, vias 32 -> 35
- net +3V3: track 39.4 -> 37.6 mm, vias 4 -> 3
- net Net-(U3-USB_DM): track 7.79 -> 8.91 mm
- net /QSPI_SS: track 10.8 -> 10.1 mm
- net Net-(U3-USB_DP): track 7.45 -> 8.02 mm
Other:
- board text added: "RP2350-V1.0"
- board text removed: "#REV 1.4"
