File: RP2350/EnvOpenPico2350/EnvOpenPico2350.kicad_sch (KiCad schematic)
At the start: 57 parts, among them J1 USB_C_Receptacle_USB2.0, J2 TSA343G00-250J2, J3 2.54mm header 01x20, J4 2.54mm header 01x20, J5 Conn_01x03_Male, Q1 SI2301B, U1 SOT-23-5 5.5V 3.3V 500mA, U2 USBLC6-2SC6, U3 RP2350A, Y1 3225_4P 12MHz

Commit message: made various corrections and adjustments to the board, generated production files.
Parts:
- D1: value 1N4002W -> 1N5917W
- FLASH1: footprint Package_SON:SON-8-1EP_3x2mm_P0.5mm_EP1.4x1.6mm -> Package_SON:Winbond_USON-8-1EP_3x2mm_P0.5mm_EP0.2x1.6mm
Other:
- note added: "Power LED is on by default but when GPIO23 is enabled it will be shut off"
- note removed: "Power LED is on by default but when GPIO24 is enabled it will be shut off"
Changed lines of the file:
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@@
 	(wire
 		(pts
-			(xy 35.56 114.3) (xy 46.99 114.3)
-		)
-		(stroke
-			(width 0)
-			(type default)
-		)
-	)
-	(wire
-		(pts
 			(xy 111.76 33.02) (xy 113.03 33.02)
 		)
@@
 	(wire
 		(pts
+			(xy 35.56 114.3) (xy 46.99 114.3)
+		)
+		(stroke
+			(width 0)
+			(type default)
+		)
+	)
+	(wire
+		(pts
 			(xy 147.32 167.64) (xy 144.78 167.64)
 		)
@@
 		)
 	)
-	(text "Power LED is on by default but when\nGPIO24 is enabled it will be shut off"
+	(text "Power LED is on by default but when\nGPIO23 is enabled it will be shut off"
 		(exclude_from_sim no)
 		(at 368.3 227.33 0)
@@
 	)
 	(label "QSPI_SS"
-		(at 38.1 114.3 0)
+		(at 35.56 114.3 0)
 		(fields_autoplaced yes)
 		(effects
@@
 		(dnp no)
 		(property "Reference" "GPIO25_LED1"
-			(at 373.38 203.2 0)
+			(at 377.825 203.835 0)
 			(effects
 				(font
@@
 			)
 		)
-		(property "Value" "1N4002W"
+		(property "Value" "1N5917W"
 			(at 72.39 27.2796 0)
 			(effects
@@
 			)
 		)
-		(property "Footprint" "Package_SON:SON-8-1EP_3x2mm_P0.5mm_EP1.4x1.6mm"
+		(property "Footprint" "Package_SON:Winbond_USON-8-1EP_3x2mm_P0.5mm_EP0.2x1.6mm"
 			(at 57.15 121.92 0)
 			(effects
@@
 		(dnp no)
 		(property "Reference" "R101"
-			(at 62.23 34.29 0)
+			(at 66.04 38.1 90)
 			(effects
 				(font
